File: data-interface-schematics/data-interface-schematics.kicad_sch (KiCad schematic)
At the start: 12 parts, among them J1 USB_A, J2 Trigger Button Input, J3 Trigger Button Wire Connector, SW1 SW_DIP_x08, SW2 SW_Push, SW3 SW_Push

Commit message: Work on schematic
Parts:
- D1: footprint LED_THT:LED_D5.0mm -> LED_THT:LED_D3.0mm
- D2: value Connected LED -> Data LED; footprint LED_THT:LED_D5.0mm -> LED_THT:LED_D3.0mm
- R1, R2: footprint Resistor_THT:R_Axial_DIN0309_L9.0mm_D3.2mm_P12.70mm_Horizontal -> Resistor_THT:R_Axial_DIN0207_L6.3mm_D2.5mm_P10.16mm_Horizontal
- SW1: footprint (none) -> Button_Switch_THT:SW_DIP_SPSTx08_Slide_9.78x22.5mm_W7.62mm_P2.54mm
- SW2: footprint (none) -> Button_Switch_THT:SW_PUSH_6mm
Changed lines of the file:
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@@
+		)
+	)
+	(text_box "Data LED should blink each time a data packet is received"
+		(exclude_from_sim no)
+		(at 228.6 93.98 0)
+		(size 21.59 10.16)
+		(stroke
+			(width 0)
+			(type default)
+		)
+		(fill
+			(type none)
+		)
+		(effects
+			(font
+				(size 1.27 1.27)
+			)
+			(justify left top)
 		)
 	)
@@
 		(exclude_from_sim no)
 		(in_bom yes)
-		(on_board yes)
+		(on_board no)
 		(dnp no)
 		(fields_autoplaced yes)
@@
 		(exclude_from_sim no)
 		(in_bom yes)
-		(on_board yes)
+		(on_board no)
 		(dnp no)
 		(property "Reference" "J3"
@@
 			)
 		)
-		(property "Footprint" ""
+		(property "Footprint" "Button_Switch_THT:SW_PUSH_6mm"
 			(at 83.82 111.76 0)
 			(effects
@@
 			)
 		)
-		(property "Footprint" "Resistor_THT:R_Axial_DIN0309_L9.0mm_D3.2mm_P12.70mm_Horizontal"
+		(property "Footprint" "Resistor_THT:R_Axial_DIN0207_L6.3mm_D2.5mm_P10.16mm_Horizontal"
 			(at 109.474 131.826 90)
 			(effects
@@
 			)
 		)
-		(property "Footprint" ""
+		(property "Footprint" "Button_Switch_THT:SW_DIP_SPSTx08_Slide_9.78x22.5mm_W7.62mm_P2.54mm"
 			(at 210.82 55.88 0)
 			(effects
@@
 			)
 		)
-		(property "Footprint" "Resistor_THT:R_Axial_DIN0309_L9.0mm_D3.2mm_P12.70mm_Horizontal"
+		(property "Footprint" "Resistor_THT:R_Axial_DIN0207_L6.3mm_D2.5mm_P10.16mm_Horizontal"
 			(at 212.344 92.964 90)
 			(effects
@@
 		(dnp no)
 		(property "Reference" "D2"
-			(at 192.659 91.7576 0)
+			(at 195.453 90.7416 0)
 			(effects
 				(font
@@
 			)
 		)
-		(property "Value" "Connected LED"
-			(at 192.659 89.2176 0)
+		(property "Value" "Data LED"
+			(at 195.453 88.2016 0)
 			(effects
 				(font
@@
 			)
 		)
-		(property "Footprint" "LED_THT:LED_D5.0mm"
+		(property "Footprint" "LED_THT:LED_D3.0mm"
 			(at 199.39 93.98 0)
 			(effects
@@
 			)
 		)
-		(property "Footprint" "LED_THT:LED_D5.0mm"
+		(property "Footprint" "LED_THT:LED_D3.0mm"
 			(at 110.49 119.38 0)
 			(effects

Commit message: Changes to schematics
Parts:
- added R3, R4: 1K, Resistor_THT:R_Axial_DIN0207_L6.3mm_D2.5mm_P10.16mm_Horizontal, symbol Device:R_US
Connections:
- net at A1.MOSI (SPI_MOSI): now also R4.1; no longer J1.2 (D-)
- net at A1.SCK (SPI_SCK): now also R3.1; no longer J1.3 (D+)
- new net: J1.3 (D+), R3.2
- new net: J1.2 (D-), R4.2
- no-connect marks 1 -> 18
Other:
- moved on the sheet: J1
