File: schematics/data-interface.kicad_sch (KiCad schematic)
At the start: 23 parts, among them J1 USB_A, J2 USB_A, J3 USB_B_Micro, J4 Trigger Button Wire Connector, J5 Trigger Button Input Connector, Q1 2SC945, Q2 2SC945, Q3 2SC945, SW1 SW_Push, SW2 SW_Push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

Commit message: Fixed minor errors in schematics
Changed lines of the file:
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@@
 		)
 	)
-	(text_box "A0-A3 and D14-D16 should have internal pull-ups enabled.\nD10 is PWM output for the buzzer.\nD9 is data LED output."
+	(text_box "A0-A2 and D14-D16 must have internal pull-ups enabled.\nD10 is PWM output for the buzzer.\nA3 is data LED output."
 		(exclude_from_sim no)
 		(at 163.83 91.44 0)
@@
 		)
 	)
-	(text_box "D7 must have pull-up resitiors enabled."
+	(text_box "D7 must have internal pull-up resitiors enabled."
 		(exclude_from_sim no)
 		(at 114.3 90.17 0)
@@
 		)
 	)
-	(text_box "J2 and J3 should use use JST connectors"
-		(exclude_from_sim no)
-		(at 93.98 123.19 0)
-		(size 20.32 7.62)
-		(stroke
-			(width 0)
-			(type default)
-		)
-		(fill
-			(type none)
-		)
-		(effects
-			(font
-				(size 1.27 1.27)
-			)
-			(justify left top)
-		)
-	)
 	(text_box "Example USB cable with trigger button capability.\nNote: The USB Micro B device is supplying power on VBUS."
 		(exclude_from_sim no)
@@
 		)
 	)
-	(text_box "The resistance between GND and all of VBUS, D+, and D- in parallel can not be less than ~4.7k before the calipers start to behave weirdly"
+	(text_box "The resistance between GND and all of VBUS, D+, and D- in parallel must not be less than ~5k ohms before the calipers start to behave weirdly"
 		(exclude_from_sim no)
 		(at 55.88 83.82 0)
-		(size 24.13 15.24)
+		(size 24.13 17.78)
 		(stroke
 			(width 0)
